File: Mux64/Mux64.kicad_sch (KiCad schematic)
At the start: 9 parts

Commit message: Add files via upload
Parts:
- gave numbers to parts that had none: 9

Commit message: Add files via upload
Other:
- note added: "ETROC Connectors"
- note removed: "RB Connectors"

Commit message: Add files via upload
Parts:
- R1, R2, R3: footprint Resistor_SMD:R_0603_1608Metric -> Resistor_SMD:R_0805_2012Metric

Commit message: Add files via upload
Parts:
- added H1, H2, H3, H4: MountingHole, MountingHole:MountingHole_2.5mm, symbol Mechanical:MountingHole
Connections:
- net scl: no longer J1.02, J2.02
- net sda: no longer J1.04, J2.04
- new net A_scl: J1.02
- new net A_sda: J1.04
- new net C_scl: J2.02
- new net C_sda: J2.04
Changed lines of the file:
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@@
     (effects (font (size 1.27 1.27)) (justify right bottom))
   )
-  (label "scl" (at 44.45 82.55 0)
+  (label "A_scl" (at 44.45 82.55 0)
     (effects (font (size 1.27 1.27)) (justify left bottom))
   )
@@
     (effects (font (size 1.27 1.27)) (justify right bottom))
   )
-  (label "scl" (at 44.45 175.26 0)
+  (label "C_scl" (at 44.45 175.26 0)
     (effects (font (size 1.27 1.27)) (justify left bottom))
   )
@@
     (effects (font (size 1.27 1.27)) (justify right bottom))
   )
-  (label "sda" (at 44.45 80.01 0)
+  (label "A_sda" (at 44.45 80.01 0)
     (effects (font (size 1.27 1.27)) (justify left bottom))
   )
@@
     (effects (font (size 1.27 1.27)) (justify right bottom))
   )
-  (label "sda" (at 44.45 172.72 0)
+  (label "C_sda" (at 44.45 172.72 0)
     (effects (font (size 1.27 1.27)) (justify left bottom))
   )
@@
     (property "Intersheet References" "${INTERSHEET_REFS}" (id 0) (at 28.7926 34.2106 0)
       (effects (font (size 1.27 1.27)) (justify right) hide)
+    )
+  )
+  (symbol (lib_id "Mechanical:MountingHole") (at 198.12 40.64 0) (unit 1)
+    (in_bom yes) (on_board yes) (fields_autoplaced)
+    (property "Reference" "H4" (id 0) (at 200.66 39.3699 0)
+      (effects (font (size 1.27 1.27)) (justify left))
+    )
+    (property "Value" "MountingHole" (id 1) (at 200.66 41.9099 0)
+      (effects (font (size 1.27 1.27)) (justify left))
+    )
+    (property "Footprint" "MountingHole:MountingHole_2.5mm" (id 2) (at 198.12 40.64 0)
+      (effects (font (size 1.27 1.27)) hide)
+    )
+    (property "Datasheet" "~" (id 3) (at 198.12 40.64 0)
+      (effects (font (size 1.27 1.27)) hide)
     )
   )
@@
     (pin "1")
   )
+  (symbol (lib_id "Mechanical:MountingHole") (at 179.07 40.64 0) (unit 1)
+    (in_bom yes) (on_board yes) (fields_autoplaced)
+    (property "Reference" "H2" (id 0) (at 181.61 39.3699 0)
+      (effects (font (size 1.27 1.27)) (justify left))
+    )
+    (property "Value" "MountingHole" (id 1) (at 181.61 41.9099 0)
+      (effects (font (size 1.27 1.27)) (justify left))
+    )
+    (property "Footprint" "MountingHole:MountingHole_2.5mm" (id 2) (at 179.07 40.64 0)
+      (effects (font (size 1.27 1.27)) hide)
+    )
+    (property "Datasheet" "~" (id 3) (at 179.07 40.64 0)
+      (effects (font (size 1.27 1.27)) hide)
+    )
+  )
   (symbol (lib_id "power:GND") (at 229.87 95.25 270) (unit 1)
     (in_bom yes) (on_board yes) (fields_autoplaced)
@@
     )
     (pin "1")
+  )
+  (symbol (lib_id "Mechanical:MountingHole") (at 198.12 31.75 0) (unit 1)
+    (in_bom yes) (on_board yes) (fields_autoplaced)
+    (property "Reference" "H3" (id 0) (at 200.66 30.4799 0)
+      (effects (font (size 1.27 1.27)) (justify left))
+    )
+    (property "Value" "MountingHole" (id 1) (at 200.66 33.0199 0)
+      (effects (font (size 1.27 1.27)) (justify left))
+    )
+    (property "Footprint" "MountingHole:MountingHole_2.5mm" (id 2) (at 198.12 31.75 0)
+      (effects (font (size 1.27 1.27)) hide)
+    )
+    (property "Datasheet" "~" (id 3) (at 198.12 31.75 0)
+      (effects (font (size 1.27 1.27)) hide)
+    )
   )
   (symbol (lib_id "power:GND") (at 38.1 54.61 270) (unit 1)
@@
     (pin "1")
   )
+  (symbol (lib_id "Mechanical:MountingHole") (at 179.07 31.75 0) (unit 1)
+    (in_bom yes) (on_board yes) (fields_autoplaced)
+    (property "Reference" "H1" (id 0) (at 181.61 30.4799 0)
+      (effects (font (size 1.27 1.27)) (justify left))
+    )
+    (property "Value" "MountingHole" (id 1) (at 181.61 33.0199 0)
+      (effects (font (size 1.27 1.27)) (justify left))
+    )
+    (property "Footprint" "MountingHole:MountingHole_2.5mm" (id 2) (at 179.07 31.75 0)
+      (effects (font (size 1.27 1.27)) hide)
+    )
+    (property "Datasheet" "~" (id 3) (at 179.07 31.75 0)
+      (effects (font (size 1.27 1.27)) hide)
+    )
+  )
   (symbol (lib_id "Device:R_Small_US") (at 35.56 160.02 90) (unit 1)
     (in_bom yes) (on_board yes) (fields_autoplaced)
@@
       (reference "C12") (unit 1) (value "0.1uF") (footprint "Capacitor_SMD:C_0805_2012Metric")
     )
+    (path "/cb7cae1e-d5f0-4217-bb9f-31ceb8262c5b"
+      (reference "H1") (unit 1) (value "MountingHole") (footprint "MountingHole:MountingHole_2.5mm")
+    )
+    (path "/256e2b56-137f-4d7f-9abf-9904299857a7"
+      (reference "H2") (unit 1) (value "MountingHole") (footprint "MountingHole:MountingHole_2.5mm")
+    )
+    (path "/37c86234-f7a7-4830-a243-0fe2831f69be"
+      (reference "H3") (unit 1) (value "MountingHole") (footprint "MountingHole:MountingHole_2.5mm")
+    )
+    (path "/0dd9a1d7-fbde-41c3-bb9f-3dab066920a2"
+      (reference "H4") (unit 1) (value "MountingHole") (footprint "MountingHole:MountingHole_2.5mm")
+    )
     (path "/7baf1f4d-513d-4881-82a8-93a37bbd2214"
       (reference "J1") (unit 1) (value "QTE-020-01-X-D-A") (footprint "QTE-020-01-X-D-A:SAMTEC_QTE-020-01-X-D-A")
@@
       (reference "R7") (unit 1) (value "1Kohm") (footprint "Resistor_SMD:R_0805_2012Metric")
     )
-    (path "/91a9abc3-7cd3-42a2-b8f1-7970bc77b6c3/4b6eec3b-f4bb-475a-803f-985d6e69cc41"
-      (reference "R8") (unit 1) (value "0ohm") (footprint "Resistor_SMD:R_0805_2012Metric")
-    )
     (path "/91a9abc3-7cd3-42a2-b8f1-7970bc77b6c3/b43b5cc7-19b3-4fa5-b538-a4d862fc3c5b/da2212cf-ed09-41e5-9780-1a165f07b1dc"
