File: Mux64_Testboard/pcb + sch files/mux64-regulators.kicad_sch (KiCad schematic)
At the start: 24 parts, among them J10 Conn_01x24, J7 Conn_01x24, J8 Conn_01x24, J9 Conn_01x24, U1 LD1117AS12TR, U2 MAX6070

Commit message: Made improvements on v1.0
Added a 100Ohm load to voltage regulator. Fixed wiring with voltage reference
Parts:
- added R24: 1Kohm, Resistor_SMD:R_0805_2012Metric, symbol Device:R_Small_US
Connections:
- net 1.2V: now also R24.2
- net B_a4: no longer C8.2, U2.6 (OUTF)
- net GND: now also R24.1
- net at R4.1, U2.5 (OUTS): now also C8.2, U2.6 (OUTF)
Changed lines of the file:
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@@
   (junction (at 107.95 48.26) (diameter 0) (color 0 0 0 0)
   )
+  (junction (at 48.26 139.7) (diameter 0) (color 0 0 0 0)
+  )
   (junction (at 118.11 143.51) (diameter 0) (color 0 0 0 0)
   )
   (junction (at 111.76 48.26) (diameter 0) (color 0 0 0 0)
   )
+  (junction (at 118.11 146.05) (diameter 0) (color 0 0 0 0)
+  )
   (junction (at 55.88 153.67) (diameter 0) (color 0 0 0 0)
   )
@@
   (junction (at 62.23 90.17) (diameter 0) (color 0 0 0 0)
   )
-  (junction (at 124.46 143.51) (diameter 0) (color 0 0 0 0)
-  )
   (junction (at 106.68 33.02) (diameter 0) (color 0 0 0 0)
   )
@@
     (stroke (width 0) (type default) (color 0 0 0 0))
   )
+  (wire (pts (xy 118.11 143.51) (xy 118.11 146.05))
+    (stroke (width 0) (type default) (color 0 0 0 0))
+  )
   (wire (pts (xy 118.11 130.81) (xy 118.11 132.08))
     (stroke (width 0) (type default) (color 0 0 0 0))
@@
     (stroke (width 0) (type default) (color 0 0 0 0))
   )
-  (wire (pts (xy 48.26 135.89) (xy 48.26 143.51))
+  (wire (pts (xy 48.26 135.89) (xy 48.26 139.7))
     (stroke (width 0) (type default) (color 0 0 0 0))
   )
@@
     (stroke (width 0) (type default) (color 0 0 0 0))
   )
-  (wire (pts (xy 124.46 143.51) (xy 124.46 146.05))
+  (wire (pts (xy 124.46 139.7) (xy 124.46 146.05))
     (stroke (width 0) (type default) (color 0 0 0 0))
   )
@@
     (stroke (width 0) (type default) (color 0 0 0 0))
   )
+  (wire (pts (xy 48.26 139.7) (xy 60.96 139.7))
+    (stroke (width 0) (type default) (color 0 0 0 0))
+  )
   (wire (pts (xy 99.06 143.51) (xy 99.06 139.7))
     (stroke (width 0) (type default) (color 0 0 0 0))
@@
     (stroke (width 0) (type default) (color 0 0 0 0))
   )
+  (wire (pts (xy 48.26 139.7) (xy 48.26 143.51))
+    (stroke (width 0) (type default) (color 0 0 0 0))
+  )
   (wire (pts (xy 99.06 163.83) (xy 118.11 163.83))
     (stroke (width 0) (type default) (color 0 0 0 0))
@@
     (stroke (width 0) (type default) (color 0 0 0 0))
   )
-  (wire (pts (xy 124.46 139.7) (xy 124.46 143.51))
-    (stroke (width 0) (type default) (color 0 0 0 0))
-  )
   (wire (pts (xy 138.43 55.88) (xy 138.43 58.42))
     (stroke (width 0) (type default) (color 0 0 0 0))
   )
+  (wire (pts (xy 60.96 148.59) (xy 55.88 148.59))
+    (stroke (width 0) (type default) (color 0 0 0 0))
+  )
   (wire (pts (xy 95.25 151.13) (xy 99.06 151.13))
     (stroke (width 0) (type default) (color 0 0 0 0))
@@
     (stroke (width 0) (type default) (color 0 0 0 0))
   )
+  (wire (pts (xy 60.96 144.78) (xy 60.96 148.59))
+    (stroke (width 0) (type default) (color 0 0 0 0))
+  )
   (wire (pts (xy 107.95 55.88) (xy 107.95 58.42))
     (stroke (width 0) (type default) (color 0 0 0 0))
@@
   )
   (wire (pts (xy 104.14 48.26) (xy 107.95 48.26))
-    (stroke (width 0) (type default) (color 0 0 0 0))
-  )
-  (wire (pts (xy 118.11 143.51) (xy 124.46 143.51))
     (stroke (width 0) (type default) (color 0 0 0 0))
   )
@@
     (pin "1")
   )
+  (symbol (lib_id "Device:R_Small_US") (at 60.96 142.24 180) (unit 1)
+    (in_bom yes) (on_board yes)
+    (property "Reference" "R24" (id 0) (at 60.96 142.24 90)
+      (effects (font (size 0.25 0.25)))
+    )
+    (property "Value" "1Kohm" (id 1) (at 59.69 142.24 90)
+      (effects (font (size 0.75 0.75)))
+    )
+    (property "Footprint" "Resistor_SMD:R_0805_2012Metric" (id 2) (at 60.96 142.24 0)
+      (effects (font (size 1.27 1.27)) hide)
+    )
+    (property "Datasheet" "~" (id 3) (at 60.96 142.24 0)
+      (effects (font (size 1.27 1.27)) hide)
+    )
+    (pin "1")
+    (pin "2")
+  )
   (symbol (lib_id "Device:R_Small_US") (at 128.27 146.05 90) (unit 1)

Commit message: Completed v2
Connections:
- net GND: no longer J9.3 (Pin_3)
- new net MUX64_A36: J9.3 (Pin_3)
